File: hardware/mu-cell-bb/mu-cell-bb.kicad_sch (KiCad schematic)
At the start: 47 parts, among them IC1 SX1255, J1 TX, J2 RX, J3 RPi Zero, U1 24LC256, U2 LDK130M33R, Y1 32MHz

Commit message: updated schematic
Parts:
- removed C7: 100n, Capacitor_SMD:C_0603_1608Metric, symbol Device:C_Small
- removed H1, H2, H3, H4: MountingHole, MountingHole:MountingHole_2.7mm_M2.5_DIN965, symbol Mechanical:MountingHole
- added C23: 100p, Capacitor_SMD:C_0603_1608Metric, symbol Device:C_Small
- added C8: 100n, Capacitor_SMD:C_0603_1608Metric, symbol Device:C_Small
- added H1, H2, H3, H4: MountingHole_M3_3.2mm_Pad, MountingHole:MountingHole_3.2mm_M3_DIN965_Pad, symbol PCM_SL_Mechanical:MountingHole_M3_3.2mm_Pad
- added J3: TX, Connector_Coaxial:U.FL_Molex_MCRF_73412-0110_Vertical, symbol Connector:Conn_Coaxial
- added J5: OLED, Connector_PinHeader_2.54mm:PinHeader_1x04_P2.54mm_Vertical, symbol PCM_SL_Pin_Headers:PINHD_1x4_Male
- added J6: IO, Connector_IDC:IDC-Header_2x06_P2.54mm_Vertical, symbol Connector_Generic:Conn_02x06_Odd_Even
- added JP1: CLK_SEL, Jumper:SolderJumper-3_P1.3mm_Bridged12_RoundedPad1.0x1.5mm_NumberLabels, symbol Jumper:Jumper_3_Bridged12
- added LED1, LED2, LED3: LED_0603, LED_SMD:LED_0603_1608Metric, symbol PCM_LED_AKL:LED_0603
- added Q1, Q2: BC817-40W, Package_TO_SOT_SMD:SOT-323_SC-70_Handsoldering, symbol PCM_Transistor_BJT_AKL:BC817-40W
- added R11, R12, R19, R20, R21, R22, R23, R24: 100R, Resistor_SMD:R_0603_1608Metric, symbol Device:R_Small
- added R13: 1M, Resistor_SMD:R_0603_1608Metric, symbol Device:R_Small
- added R14, R15, R16, R17, R18: 1K, Resistor_SMD:R_0603_1608Metric, symbol Device:R_Small
- J4: renamed from J3; value RPi Zero -> RPi GPIO
- renumbered C8 to C7
Connections:
- net +3V3: now also J6.1 (Pin_1)
- net +5V: now also J5.3, J6.2 (Pin_2), R14.1, R15.1, R17.1
- net GND: now also C10.1, C9.1, C8.1, H1.1, H2.1, H3.1, H4.1, J3.2 (Ext), J5.4, J6.11 (Pin_11), J6.12 (Pin_12), LED1.1 (K), Q1.2 (E), Q2.2 (E), R13.2; no longer C10.2, C9.2
- net TCXO_CLK: now also JP1.1 (A); no longer IC1.8 (XTB)
- net at IC1.5 (VR_DIG): now also C10.2; no longer C10.1
- net at IC1.1 (VR_PA): now also C8.2
- net RXD: now reaches J4.10 (Pin_10)
- net RXD: now also R20.1
- net GPIO17: now reaches J4.11 (Pin_11)
- net GPIO17: now also J4.36 (Pin_36), R24.1
- net GPIO27: now reaches J4.13 (Pin_13)
- net TX_EN: now reaches J4.15 (Pin_15)
- net TX_EN: now also R12.1, R16.2
- net RX_EN: now reaches J4.16 (Pin_16)
- net RX_EN: now also R11.1, R18.2
- net GPIO24: now reaches J4.18 (Pin_18)
- net GPIO25: now reaches J4.22 (Pin_22)
- net GPIO07: now reaches J4.26 (Pin_26)
- net SDA: now reaches J4.3 (Pin_3)
- net SDA: now also J5.1, R21.1
- net GPIO06: now reaches J4.31 (Pin_31)
- net GPIO12: now reaches J4.32 (Pin_32)
- net GPIO13: now reaches J4.33 (Pin_33)
- net GPIO26: now reaches J4.37 (Pin_37)
- net SCL: now reaches J4.5 (Pin_5)
- net SCL: now also J5.2, R23.1
- net GPIO04: now reaches J4.7 (Pin_7)
- net GPIO04: now also R19.1
- net TXD: now reaches J4.8 (Pin_8)
- net TXD: now also R22.1
- net at IC1.3 (VR_ANAI): now also C9.2; no longer C9.1
- net OUT renamed CK_OUT
- new net: J6.9 (Pin_9), R19.2
- new net: Q1.1 (B), R16.1
- new net: LED2.1 (K), Q1.3 (C)
- new net: LED1.2 (A), R14.2
- new net: Q2.1 (B), R18.1
- new net: LED3.1 (K), Q2.3 (C)
- new net: C23.1, J3.1 (In), R13.1
- new net: LED3.2 (A), R17.2
- new net: J6.8 (Pin_8), R23.2
- new net: J6.3 (Pin_3), R11.2
- new net: J6.10 (Pin_10), R24.2
- new net: J6.6 (Pin_6), R22.2
- new net: LED2.2 (A), R15.2
- new net: J6.7 (Pin_7), R21.2
- new net: J6.5 (Pin_5), R20.2
- new net: J6.4 (Pin_4), R12.2
- new net EXT_CLK: C23.2, JP1.3 (B)
- new net SX_CLK: IC1.8 (XTB), JP1.2 (C)
- no-connect marks 26 -> 9
Other:
- company: Jankyneering -> jankyneering.cc
- moved on the sheet: C11, C12, C14, C15, C17, C18, C19, C20, C21, C22, IC1, J1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

Commit message: started work on PCB
Parts:
- removed J5: OLED, Connector_PinHeader_2.54mm:PinHeader_1x04_P2.54mm_Vertical, symbol PCM_SL_Pin_Headers:PINHD_1x4_Male
- added OLED1: SSD1306, OLED_128x64:128x64OLED, symbol OLED_128x64:SSD1306
- J3: value TX -> EXT_CLK
- renumbered J6 to J5
Connections:
- net +5V: now also OLED1.2 (VCC)
- net GND: now also OLED1.1 (GND)
- net SCL: now also OLED1.3 (SCL)
- net SDA: now also OLED1.4 (SDA)
Changed lines of the file:
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@@
 	)
 	(symbol
-		(lib_id "power:GND")
-		(at 106.68 91.44 0)
+		(lib_id "OLED_128x64:SSD1306")
+		(at 252.73 33.02 90)
 		(unit 1)
 		(exclude_from_sim no)
@@
 		(on_board yes)
 		(dnp no)
-		(fields_autoplaced yes)
-		(property "Reference" "#PWR012"
-			(at 106.68 97.79 0)
+		(property "Reference" "OLED1"
+			(at 255.27 37.338 0)
 			(effects
 				(font
 					(size 1.27 1.27)
 				)
-				(hide yes)
+				(justify left)
 			)
 		)
-		(property "Value" "GND"
-			(at 106.68 95.5731 0)
+		(property "Value" "SSD1306"
+			(at 257.81 37.338 0)
 			(effects
 				(font
 					(size 1.27 1.27)
 				)
+				(justify left)
 			)
 		)
-		(property "Footprint" ""
-			(at 106.68 91.44 0)
+		(property "Footprint" "OLED_128x64:128x64OLED"
+			(at 246.38 33.02 0)
 			(effects
 				(font
@@
 		)
 		(property "Datasheet" ""
-			(at 106.68 91.44 0)
+			(at 246.38 33.02 0)
 			(effects
 				(font
@@
 			)
 		)
-		(property "Description" "Power symbol creates a global label with name \"GND\" , ground"
-			(at 106.68 91.44 0)
+		(property "Description" "SSD1306 OLED"
+			(at 252.73 33.02 0)
 			(effects
 				(font
@@
 		(pin "1"
 		)
+		(pin "4"
+		)
+		(pin "3"
+		)
+		(pin "2"
+		)
 		(instances
-			(project "mu-cell-bb"
+			(project ""
 				(path "/564c8f3e-4a0a-4bb3-921f-1318a09780f9"
-					(reference "#PWR012")
+					(reference "OLED1")
 					(unit 1)
 				)
@@
 	)
 	(symbol
-		(lib_id "PCM_SL_Mechanical:MountingHole_M3_3.2mm_Pad")
-		(at 148.59 181.61 0)
+		(lib_id "power:GND")
+		(at 106.68 91.44 0)
 		(unit 1)
 		(exclude_from_sim no)
@@
 		(dnp no)
 		(fields_autoplaced yes)
-		(property "Reference" "H3"
-			(at 152.4 180.3399 0)
+		(property "Reference" "#PWR012"
+			(at 106.68 97.79 0)
 			(effects
 				(font
 					(size 1.27 1.27)
 				)
-				(justify left)
+				(hide yes)
 			)
 		)
-		(property "Value" "MountingHole_M3_3.2mm_Pad"
-			(at 152.4 182.8799 0)
+		(property "Value" "GND"
+			(at 106.68 95.5731 0)
 			(effects
 				(font
 					(size 1.27 1.27)
 				)
-				(justify left)
-				(hide yes)
 			)
 		)
-		(property "Footprint" "MountingHole:MountingHole_3.2mm_M3_DIN965_Pad"
-			(at 148.59 185.42 0)
+		(property "Footprint" ""
+			(at 106.68 91.44 0)
 			(effects
 				(font
@@
 		)
 		(property "Datasheet" ""
-			(at 148.59 181.61 0)
+			(at 106.68 91.44 0)
 			(effects
 				(font
@@
 			)
 		)
-		(property "Description" "3.2mm Diameter Mounting Hole Pad (M3)"
-			(at 148.59 181.61 0)
+		(property "Description" "Power symbol creates a global label with name \"GND\" , ground"
+			(at 106.68 91.44 0)
 			(effects
 				(font
@@
 			(project "mu-cell-bb"
 				(path "/564c8f3e-4a0a-4bb3-921f-1318a09780f9"
-					(reference "H3")
+					(reference "#PWR012")
 					(unit 1)
 				)
@@
 	)
 	(symbol
-		(lib_id "PCM_SL_Pin_Headers:PINHD_1x4_Male")
-		(at 247.65 33.02 0)
+		(lib_id "PCM_SL_Mechanical:MountingHole_M3_3.2mm_Pad")
+		(at 148.59 181.61 0)
 		(unit 1)
 		(exclude_from_sim no)
@@
 		(dnp no)
 		(fields_autoplaced yes)
-		(property "Reference" "J5"
-			(at 247.525 22.86 0)
+		(property "Reference" "H3"
+			(at 152.4 180.3399 0)
 			(effects
 				(font
 					(size 1.27 1.27)
 				)
+				(justify left)
 			)
 		)
-		(property "Value" "OLED"
-			(at 247.525 25.4 0)
+		(property "Value" "MountingHole_M3_3.2mm_Pad"
+			(at 152.4 182.8799 0)
 			(effects
 				(font
 					(size 1.27 1.27)
 				)
+				(justify left)
+				(hide yes)
 			)
 		)
-		(property "Footprint" "Connector_PinHeader_2.54mm:PinHeader_1x04_P2.54mm_Vertical"
-			(at 246.38 21.59 0)
+		(property "Footprint" "MountingHole:MountingHole_3.2mm_M3_DIN965_Pad"
+			(at 148.59 185.42 0)
 			(effects
 				(font
@@
 		)
 		(property "Datasheet" ""
-			(at 247.65 22.86 0)
+			(at 148.59 181.61 0)
 			(effects
 				(font
@@
 			)
 		)
-		(property "Description" "Pin Header male with pin space 2.54mm. Pin Count -4"
-			(at 247.65 33.02 0)
+		(property "Description" "3.2mm Diameter Mounting Hole Pad (M3)"
+			(at 148.59 181.61 0)
 			(effects
 				(font
@@
 		(pin "1"
 		)
-		(pin "2"
-		)
-		(pin "3"
-		)
-		(pin "4"
-		)
 		(instances
-			(project ""
+			(project "mu-cell-bb"
 				(path "/564c8f3e-4a0a-4bb3-921f-1318a09780f9"
-					(reference "J5")
+					(reference "H3")
 					(unit 1)
 				)
@@
 			)
 		)
-		(property "Value" "TX"
+		(property "Value" "EXT_CLK"
 			(at 27.9399 34.5253 0)
 			(effects
@@
 		(dnp no)
 		(fields_autoplaced yes)
-		(property "Reference" "J6"
+		(property "Reference" "J5"
 			(at 248.92 58.42 0)
 			(effects
@@
 			(project ""
 				(path "/564c8f3e-4a0a-4bb3-921f-1318a09780f9"
-					(reference "J6")
+					(reference "J5")
 					(unit 1)
 				)

Commit message: added symbols, worked on PCB
Parts:
- removed OLED1: SSD1306, OLED_128x64:128x64OLED, symbol OLED_128x64:SSD1306
- removed U2: LDK130M33R, SOT23-5L_1P75X3P05X0P95_STM, symbol ldk130m33r:LDK130M33R
- added OLED1: SSD1306, parts:OLED_128x64_I2C, symbol parts:SSD1306
- added U2: LDK130M33R, parts:SOT23-5L_1P75X3P05X0P95_STM, symbol parts:LDK130M33R
Connections:
- net +3V3: now also U2.5 (OUT)
- net +5V: now also OLED1.2 (VCC), U2.1 (IN), U2.3 (EN)
- net GND: now also OLED1.1 (GND), U2.2 (GND)
- net SCL: now also OLED1.3 (SCL)
- net SDA: now also OLED1.4 (SDA)
- net at C21.1: now also U2.4 (BYP/ADJ)
Changed lines of the file:
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@@
 	)
 	(junction
-		(at 118.11 143.51)
-		(diameter 0)
-		(color 0 0 0 0)
-	)
-	(junction
 		(at 102.87 31.75)
 		(diameter 0)
@@
 	)
 	(junction
+		(at 118.11 143.51)
+		(diameter 0)
+		(color 0 0 0 0)
+	)
+	(junction
 		(at 240.03 154.94)
 		(diameter 0)
@@
 	)
 	(symbol
-		(lib_id "OLED_128x64:SSD1306")
-		(at 252.73 33.02 90)
-		(unit 1)
-		(exclude_from_sim no)
-		(in_bom yes)
-		(on_board yes)
-		(dnp no)
-		(property "Reference" "OLED1"
-			(at 255.27 37.338 0)
-			(effects
-				(font
-					(size 1.27 1.27)
-				)
-				(justify left)
-			)
-		)
-		(property "Value" "SSD1306"
-			(at 257.81 37.338 0)
-			(effects
-				(font
-					(size 1.27 1.27)
-				)
-				(justify left)
-			)
-		)
-		(property "Footprint" "OLED_128x64:128x64OLED"
-			(at 246.38 33.02 0)
-			(effects
-				(font
-					(size 1.27 1.27)
-				)
-				(hide yes)
-			)
-		)
-		(property "Datasheet" ""
-			(at 246.38 33.02 0)
-			(effects
-				(font
-					(size 1.27 1.27)
-				)
-				(hide yes)
-			)
-		)
-		(property "Description" "SSD1306 OLED"
-			(at 252.73 33.02 0)
-			(effects
-				(font
-					(size 1.27 1.27)
-				)
-				(hide yes)
-			)
-		)
-		(pin "1"
-		)
-		(pin "4"
-		)
-		(pin "3"
-		)
-		(pin "2"
-		)
-		(instances
-			(project ""
-				(path "/564c8f3e-4a0a-4bb3-921f-1318a09780f9"
-					(reference "OLED1")
-					(unit 1)
-				)
-			)
-		)
-	)
-	(symbol
 		(lib_id "power:GND")
 		(at 106.68 91.44 0)
@@
 	)
 	(symbol
+		(lib_id "parts:SSD1306")
+		(at 252.73 33.02 90)
+		(unit 1)
+		(exclude_from_sim no)
+		(in_bom yes)
+		(on_board yes)
+		(dnp no)
+		(property "Reference" "OLED1"
+			(at 255.016 37.592 0)
+			(effects
+				(font
+					(size 1.27 1.27)
+				)
+				(justify left)
+			)
+		)
+		(property "Value" "SSD1306"
+			(at 257.556 37.592 0)
+			(effects
+				(font
+					(size 1.27 1.27)
+				)
+				(justify left)
+			)
+		)
+		(property "Footprint" "parts:OLED_128x64_I2C"
+			(at 246.38 33.02 0)
+			(effects
+				(font
+					(size 1.27 1.27)
+				)
+				(hide yes)
+			)
+		)
+		(property "Datasheet" ""
+			(at 246.38 33.02 0)
+			(effects
+				(font
+					(size 1.27 1.27)
+				)
+				(hide yes)
+			)
+		)
+		(property "Description" "SSD1306 OLED"
+			(at 252.73 33.02 0)
+			(effects
+				(font
+					(size 1.27 1.27)
+				)
+				(hide yes)
+			)
+		)
+		(pin "2"
+		)
+		(pin "1"
+		)
+		(pin "4"
+		)
+		(pin "3"
+		)
+		(instances
+			(project ""
+				(path "/564c8f3e-4a0a-4bb3-921f-1318a09780f9"
+					(reference "OLED1")
+					(unit 1)
+				)
+			)
+		)
+	)
+	(symbol
 		(lib_id "power:GND")
 		(at 146.05 156.21 0)
@@
 	)
 	(symbol
-		(lib_id "ldk130m33r:LDK130M33R")
-		(at 127 146.05 0)
-		(unit 1)
-		(exclude_from_sim no)
-		(in_bom yes)
-		(on_board yes)
-		(dnp no)
-		(fields_autoplaced yes)
-		(property "Reference" "U2"
-			(at 127 137.16 0)
-			(effects
-				(font
-					(size 1.524 1.524)
-				)
-			)
-		)
-		(property "Value" "LDK130M33R"
-			(at 127 139.7 0)
-			(effects
-				(font
-					(size 1.524 1.524)
-				)
-			)
-		)
-		(property "Footprint" "SOT23-5L_1P75X3P05X0P95_STM"
-			(at 127 155.956 0)
-			(effects
-				(font
-					(size 1.27 1.27)
-					(italic yes)
-				)
-				(hide yes)
-			)
-		)
-		(property "Datasheet" "https://www.st.com/resource/en/datasheet/ldk130.pdf"
-			(at 127 158.242 0)
-			(effects
-				(font
-					(size 1.27 1.27)
-					(italic yes)
-				)
-				(hide yes)
-			)
-		)
-		(property "Description" ""
-			(at 127 146.05 0)
-			(effects
-				(font
-					(size 1.27 1.27)
-				)
-				(hide yes)
-			)
-		)
-		(pin "1"
-		)
-		(pin "2"
-		)
-		(pin "5"
-		)
-		(pin "4"
-		)
-		(pin "3"
-		)
-		(instances
-			(project ""
-				(path "/564c8f3e-4a0a-4bb3-921f-1318a09780f9"
-					(reference "U2")
-					(unit 1)
-				)
-			)
-		)
-	)
-	(symbol
 		(lib_id "power:+3V3")
 		(at 29.21 133.35 0)
@@
 					(unit 1)
 				)
+			)
+		)
+	)
+	(symbol
+		(lib_id "parts:LDK130M33R")
+		(at 127 146.05 0)
+		(unit 1)
+		(exclude_from_sim no)
+		(in_bom yes)
+		(on_board yes)
+		(dnp no)
+		(fields_autoplaced yes)
+		(property "Reference" "U2"
+			(at 127 135.89 0)
+			(effects
+				(font
+					(size 1.524 1.524)
+				)
+			)
+		)
+		(property "Value" "LDK130M33R"
+			(at 127 138.43 0)
+			(effects
+				(font
+					(size 1.524 1.524)
+				)
+			)
+		)
+		(property "Footprint" "parts:SOT23-5L_1P75X3P05X0P95_STM"
+			(at 127 159.512 0)
+			(effects
+				(font
+					(size 1.27 1.27)
+					(italic yes)
+				)
+				(hide yes)
+			)
+		)
+		(property "Datasheet" "https://www.st.com/resource/en/datasheet/ldk130.pdf"
+			(at 126.492 163.576 0)
+			(effects
+				(font
+					(size 1.27 1.27)
+					(italic yes)
+				)
+				(hide yes)
+			)
+		)
+		(property "Description" ""
+			(at 127 146.05 0)
+			(effects
+				(font
+					(size 1.27 1.27)
+				)
+				(hide yes)
+			)
+		)
+		(pin "1"
+		)
+		(pin "4"
+		)
+		(pin "5"
+		)
+		(pin "2"
+		)
+		(pin "3"
+		)
+		(instances
+			(project ""
+				(path "/564c8f3e-4a0a-4bb3-921f-1318a09780f9"
+					(reference "U2")
+					(unit 1)
+				)

Commit message: added parts
Parts:
- removed J1: TX, Connector_Coaxial:U.FL_Molex_MCRF_73412-0110_Vertical, symbol Connector:Conn_Coaxial
- removed J2: RX, Connector_Coaxial:U.FL_Molex_MCRF_73412-0110_Vertical, symbol Connector:Conn_Coaxial
- removed J3: EXT_CLK, Connector_Coaxial:U.FL_Molex_MCRF_73412-0110_Vertical, symbol Connector:Conn_Coaxial
- added J1: TX, parts:U.FL_Vertical_Passthrough, symbol parts:Conn_Coaxial
- added J2: RX, parts:U.FL_Vertical_Passthrough, symbol parts:Conn_Coaxial
- added J3: EXT_CLK, symbol parts:Conn_Coaxial
- added JSMA1: TX, parts:BATWIRELESS_BWSMA-KE-P001, symbol parts:Conn_Coaxial
- added JSMA2: RX, parts:BATWIRELESS_BWSMA-KE-P001, symbol parts:Conn_Coaxial
Connections:
- net GND: now also J1.2 (Ext), J2.2 (Ext), J3.2 (Ext), JSMA1.2 (Ext), JSMA2.2 (Ext)
- net at L2.1: now also J2.1 (In), JSMA2.1 (In)
- net at C23.1, R13.1: now also J3.1 (In)
- net at C14.1, L3.2: now also J1.1 (In), JSMA1.1 (In)
