File: hardware/mu-cell-bb/mu-cell-bb.kicad_sch (KiCad schematic)
At the start: 81 parts, among them IC1 SX1255IWLTRT, J1 TX, J2 RX, J3 EXT_CLK, J4 RPi GPIO, J5 IO, J6 TC2030, J7 TC2030, Q1 BC817-40W, Q2 BC817-40W, U1 24LC256, U2 LDK130M33R, Y1 38.4MHz

Commit message: added v1.3 files
Parts:
- C1, C2: MPN (none) -> GCM1555C1H101FA16D
- C10, C11, C12, C14, C16, C21, C24, C7, C9: MPN 06035G104ZAT2A -> CC0402KRX7R7BB104
- C13, C15, C17, C18, C19, C22: MPN C0603C103M4REC7411 -> CC0402KRX7R9BB103
- C20, C23: MPN 06035G104ZAT2A -> CL05A105KO5NNNC
- C25: MPN 06035G104ZAT2A -> CL05A475MP5NRNC
- C3: MPN (none) -> GCM1555C1H3R3GA16D
- C4: MPN (none) -> 0402CG8R2G500NT
- C5: MPN (none) -> GCM1555C1H6R8FA16D
- C6, C8: MPN 06035G104ZAT2A -> GCM1555C1H101FA16D
- D1: MPN (none) -> BAV99,215
- IC1: MPN (none) -> SX1255IWLTRT
- J1, J2, J3: MPN (none) -> BWU.FL-IPEX1
- L1, L3, L4: MPN (none) -> 0402CS-39NXGRW
- L2: MPN (none) -> 0402CS-22NXGRW
- LED1: MPN (none) -> F.0402.00003/P2-0402R1TS2-045T-001
- LED2: MPN (none) -> BL-HJC37A-AV-TRB
- LED3: MPN (none) -> 16-213/GHC-YR1S1/3T
- Q1, Q2: MPN (none) -> LBC817-40WT1G
- R1, R19, R2, R20, R21, R22, R23, R24, R25, R26, R3, R4, R5, R6, R7: MPN CRCW0603100RFKECC -> RC0402FR-07100RL
- R10, R8, R9: MPN CRCW0603100RFKECC -> 0402WGF1004TCE
- R11, R12, R13: MPN CRCW06033K9FKECC -> FRC0402F3901TS
- R14, R15, R16, R17, R18: MPN CRCW06033K9FKECC -> RC0402FR-071KL
- RFCAN1: MPN (none) -> 2118707-4
- U1: MPN (none) -> 24LC256-E/SN
- U2: MPN (none) -> LDK130M33R
- Y1: MPN (none) -> TG2016SMN 38.4000M-MCGNNM3
Connections:
- net +3V3: no longer J5.1 (Pin_1)
- net +3V3_PI: now reaches J4.1 (Pin_1)
- net +3V3_PI: now also J5.1 (Pin_1)
- no-connect marks 9 -> 8
