File: hardware/mu-cell-bb/mu-cell-bb.kicad_pcb (KiCad board)
At the start: 4 copper layers, 65 x 30 mm, 83 parts, among them IC1 SX1255IWLTRT, J1 TX, J2 RX, J3 EXT_CLK, J4 RPi GPIO, J5 IO, J6 TC2030, J7 TC2030, Q1 BC817-40W, Q2 BC817-40W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

Commit message: added v1.2 PCB files
Parts:
- added ?: , clipboard:e7774905-3e1b-474f-b2b7-99bac235eba3, F.Cu at (149.3, 101.0)
- added ?: , clipboard:e7774905-3e1b-474f-b2b7-99bac235eba3, F.Cu at (148.9, 97.7)
- Y1: footprint parts:Oscillator_SMD_ECS_2520MV-xxx-xx-4Pin_2.5x2.0mm -> Crystal:Crystal_SMD_2016-4Pin_2.0x1.6mm
- turned Y1 to -90 degrees
