File: hardware/mu-cell-bb/mu-cell-bb.kicad_pcb (KiCad board)
At the start: 4 copper layers, 65 x 30 mm, 85 parts, among them IC1 SX1255IWLTRT, J1 TX, J2 RX, J3 EXT_CLK, J4 RPi GPIO, J5 IO, J6 TC2030, J7 TC2030, Q1 BC817-40W, Q2 BC817-40W, U1 24LC256, U2 LDK130M33R, Y1 38.4MHz

Commit message: added v1.3 files
Connections:
- J4 pad 1: unconnected-(J4-Pin_1-Pad1) -> +3V3_PI
- J5 pad 1: +3V3 -> +3V3_PI
Routing:
- net +3V3: track 109.8 -> 80.1 mm
- net +3V3_PI: track 0.00 -> 18.0 mm
- net GND: track 24.1 -> 26.6 mm
- net /SDA: track 29.6 -> 30.2 mm
